File: pcb/pcb_01/pcb_01.kicad_pcb (KiCad board)
At the start: 2 copper layers, 2 parts, among them J1 Screw_Terminal_01x02

Commit message: update pcb
Parts:
- added J2: Screw_Terminal_01x03, TerminalBlock:TerminalBlock_bornier-3_P5.08mm, F.Cu at (127.0, 111.8)
- added J3: Screw_Terminal_01x02, TerminalBlock:TerminalBlock_bornier-2_P5.08mm, F.Cu at (144.8, 76.2)
- added RV1: R_Potentiometer, Potentiometer_THT:Potentiometer_Alps_RK097_Single_Horizontal, F.Cu at (144.8, 111.8)
- added U1: LM358, Package_DIP:DIP-8_W7.62mm, F.Cu at (151.1, 90.2)
- moved RZ1 5.24 mm to (136.6, 102.9)
- moved J1 2.54 mm to (121.9, 76.2)
Connections:
- J1 pad 1: Net-(RZ1-Pad23) -> Net-(RZ1-Pad7)
- J1 pad 2: Net-(RZ1-Pad6) -> Net-(RZ1-Pad23)
- RZ1 pad 17: unconnected-(RZ1-Pad17) -> Net-(RZ1-Pad17)
- RZ1 pad 18: unconnected-(RZ1-Pad18) -> Net-(RZ1-Pad18)
- RZ1 pad 21: unconnected-(RZ1-Pad21) -> Net-(RZ1-Pad21)
- RZ1 pad 22: unconnected-(RZ1-Pad22) -> Net-(RZ1-Pad22)
- RZ1 pad 6: Net-(RZ1-Pad6) -> unconnected-(RZ1-Pad6)
- RZ1 pad 7: unconnected-(RZ1-Pad7) -> Net-(RZ1-Pad7)
- RZ1 pad 9: unconnected-(RZ1-Pad9) -> Net-(RZ1-Pad9)
Routing:
- net Net-(RZ1-Pad23): track 0.00 -> 101.6 mm
- net Net-(RZ1-Pad22): track 0.00 -> 49.1 mm
- net Net-(RZ1-Pad21): track 0.00 -> 31.0 mm
- net Net-(RZ1-Pad17): track 0.00 -> 23.1 mm
- net Net-(U1-Pad1): track 0.00 -> 17.0 mm
- net Net-(RZ1-Pad7): track 0.00 -> 13.4 mm
- net Net-(RZ1-Pad9): track 0.00 -> 12.6 mm
- net Net-(RZ1-Pad18): track 0.00 -> 10.4 mm
- net (no net): vias 5 -> 0
Other:
- board outline added: 43.2 x 45.7 mm

Commit message: update
Routing:
- net Net-(J2-Pad1): track 10.4 -> 0.57 mm
- net Net-(J1-Pad2): track 101.6 -> 95.0 mm
- net Net-(RV1-Pad1): track 31.0 -> 29.2 mm
Other:
- board size 43.2 x 45.7 mm -> 45.7 x 45.7 mm

Commit message: update pcb
Parts:
- added RV2: R_Potentiometer, Potentiometer_THT:Potentiometer_Alps_RK097_Single_Horizontal, F.Cu at (167.6, 128.2)
- RZ1: value RP2040-Zero -> RP2040-Zero_1; footprint rp2040-zero:RP2040-Zero -> rp2040-zero:RP2040-Zero_copia
- moved J1 67.7 mm to (188.0, 91.3), turned to -90 degrees
- moved J2 61.2 mm to (188.0, 116.7), turned to -90 degrees
- moved J3 51.4 mm to (188.0, 104.1), turned to -90 degrees
- moved RV1 19.3 mm to (134.6, 128.2)
- moved U1 18.3 mm to (166.4, 100.3)
- moved RZ1 16.1 mm to (141.7, 118.1)
Connections:
- net Net-(J1-Pad2) renamed Earth
- J2 pad 1: Net-(J2-Pad1) -> Net-(RZ1-Pad19)
- RZ1 pad 17: Net-(RV1-Pad2) -> Net-(RZ1-Pad17)
- RZ1 pad 18: Net-(J2-Pad1) -> Net-(RV1-Pad2)
- RZ1 pad 19: unconnected-(RZ1-Pad19) -> Net-(RZ1-Pad19)
Routing:
- net Earth: track 95.0 -> 0.00 mm
- net Net-(RZ1-Pad19): track 0.00 -> 60.0 mm
- net Net-(J1-Pad1): track 13.4 -> 57.2 mm
- net Net-(J2-Pad3): track 49.1 -> 89.9 mm
- net Net-(RZ1-Pad17): track 0.00 -> 40.2 mm
- net Net-(RV1-Pad1): track 29.2 -> 15.5 mm
- net Net-(RV1-Pad2): track 23.1 -> 13.4 mm
- net Net-(U1-Pad3): track 12.6 -> 21.7 mm
- net Net-(J3-Pad2): track 17.0 -> 25.3 mm
- net Net-(J2-Pad1): track 0.57 -> 0.00 mm
- added copper zone on B.Cu, net Earth
Other:
- board size 45.7 x 45.7 mm -> 76.2 x 45.7 mm

Commit message: update pcb
Parts:
- moved RV1 1.22 mm to (134.6, 127.0)
- moved RV2 1.22 mm to (167.6, 127.0)
Connections:
- J2 pad 1: Net-(RZ1-Pad19) -> Earth
- J2 pad 2: Earth -> Net-(RZ1-Pad19)
Routing:
- net Net-(RV1-Pad1): track 15.5 -> 49.4 mm
- net Net-(RZ1-Pad9): track 21.7 -> 26.5 mm
- net Net-(J3-Pad2): track 25.3 -> 27.8 mm
- net Net-(RZ1-Pad19): track 60.0 -> 62.1 mm
- net Net-(RV2-Pad2): track 40.2 -> 42.1 mm
- net Net-(J1-Pad1): track 57.2 -> 58.8 mm
- net Net-(J2-Pad3): track 89.9 -> 91.5 mm
- net Net-(RV1-Pad2): track 13.4 -> 12.2 mm
